File: A2BFeatherWing_A2B.sch (KiCad schematic (older format))
At the start: 71 parts, among them Q1 Q_PMOS_GDS, U1 AD2428W

Commit message: added 3d model of JST PH and CM added eco layer for silkscreen
Parts:
- removed C76, C77: 3n3, symbol Device:C_Small
- removed FB3 (x2), FB4 (x2): L_Small, symbol Device:L_Small
- removed JP?: SolderJumper_2_Bridged, symbol Jumper:SolderJumper_2_Open
- removed R? (x2): 10k, symbol Device:R_Small
- added C15, C6: 0u1, Capacitor_SMD:C_0402_1005Metric, symbol Device:C_Small
- added C41: 10u, Capacitor_SMD:C_0805_2012Metric, symbol Device:C_Small
- C1: renamed from C?; footprint (none) -> Capacitor_SMD:C_0402_1005Metric
- C12, C13, C14, C18, C51, C52, C55, C57, C60, C70, C71, C74, C75, C8, C86, C87, C88, C89, C9: footprint (none) -> Capacitor_SMD:C_0402_1005Metric
- C2, C3: renamed from C?; footprint (none) -> Capacitor_SMD:C_0603_1608Metric
- C20, C21, C4, C5, C56, C58: footprint (none) -> Capacitor_SMD:C_0603_1608Metric
- C30: footprint (none) -> Capacitor_SMD:C_0805_2012Metric
- C53: renamed from C88; footprint (none) -> Capacitor_SMD:C_0402_1005Metric
- C54: renamed from C89; footprint (none) -> Capacitor_SMD:C_0402_1005Metric
- C7: value 33n -> 0u47; footprint (none) -> Capacitor_SMD:C_0603_1608Metric
- C72: value 3n3 -> 12p; footprint (none) -> Capacitor_SMD:C_0402_1005Metric
- C73: renamed from C?; value 3n3 -> 12p; footprint (none) -> Capacitor_SMD:C_0402_1005Metric
- CM1: renamed from CM2; footprint Knochi_Filters:CommonModeChoke_TDK_ACT1210 -> A2BFeatherWing:CommonModeChoke_TDK_ACT1210
- CM2: footprint Knochi_Filters:CommonModeChoke_TDK_ACT1210 -> A2BFeatherWing:CommonModeChoke_TDK_ACT1210
- D1, D2: footprint (none) -> Diode_SMD:D_SOD-523
- D3: footprint (none) -> Diode_SMD:D_SOD-123
- JP1, JP2: renamed from JP?; footprint (none) -> Jumper:SolderJumper-3_P1.3mm_Bridged12_Pad1.0x1.5mm
- L1, L2, L3, L4: footprint (none) -> Inductor_SMD:L_0402_1005Metric
- L5, L6, L7, L8: footprint (none) -> Inductor_SMD:L_0805_2012Metric
- Q1: footprint (none) -> Package_TO_SOT_SMD:SOT-23
- R1, R2, R3, R4, R8: footprint (none) -> Resistor_SMD:R_0603_1608Metric
- R11, R13: renamed from R?; footprint (none) -> Resistor_SMD:R_0402_1005Metric
- R5, R6, R7: footprint (none) -> Resistor_SMD:R_0402_1005Metric
- R9: footprint (none) -> Resistor_SMD:R_0805_2012Metric
Connections:
- net +3V3: now also JP1.3 (B), JP2.3 (B), C15.1
- net GND: now also JP1.1 (A), JP2.1 (A), C15.2, C41.2, C6.2; no longer R11.2, R13.2
- net IO1: now also R11.2; no longer JP1.2 (C)
- net IO2: now also R13.1; no longer JP2.2 (C)
- net VIN: now also C41.1, C6.1
- net B''P: now reaches C86.2, L1.1
- net B''P: now also CM1.3; no longer CM1.1
- net B'P: now reaches C2.2, R1.1
- net B'P: now also CM1.4; no longer CM1.2
- net B''N: now reaches C87.1, L2.2
- net B''N: now also CM1.1; no longer CM1.3
- net B'N: now reaches C3.2, R2.2
- net B'N: now also CM1.2; no longer CM1.4
- net B'''P: now reaches C72.1, L1.2, U1.22 (BP)
- net B'''N: now reaches C72.2, L2.1, U1.23 (BN)
- net A''P: now reaches C88.2, CM2.1, L3.1
- net A'P: now reaches C4.2, CM2.2, R3.1
- net A''N: now reaches C89.1, CM2.3, L4.2
- net A'N: now reaches C5.2, CM2.4, R4.2
- net A'''N: now reaches C73.2, L4.1, U1.18 (AN)
- net A'''P: now reaches C73.1, L3.2, U1.19 (AP)
- net at R11.1: now also JP1.2 (C); no longer JP1.1 (A)
- net IO0 renamed IRQ
- net IO3 renamed DTX0
- net IO4 renamed DTX1
- net IO5 renamed DRX0
- net IO6 renamed DRX1
- new net: JP2.2 (C), R13.2
Other:
- note added: "EMC Filter \nfor FM and DAB bands"
- note added: "EMC Notch Filter\n"
- moved on the sheet: C1, C2, C3, C30, C4, C5, C51, C52, C53, C54, C60, C7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

Commit message: last changes
Other:
- note added: "EMC Notch Filter\n(not on PCB)\n"
- note removed: "EMC Notch Filter\n"
Changed lines of the file:
@@
 Wire Notes Line
 	5150 5800 5150 3675
-Text Notes 5125 5900 0    50   ~ 0
-EMC Notch Filter\n
+Text Notes 5125 5975 0    50   ~ 0
+EMC Notch Filter\n(not on PCB)\n
 Text Label 7675 3850 0    50   ~ 0
 B'P
